File: atividades/atividade-03/controlador_temperatura.sch (EAGLE design)
At the start: 10 parts, among them Q1 BC337

Commit message: pump scheme
Parts:
- added D2: 1N4007, diode:1N4004
- added PUMP: MKDSN1,5/2-5,08, con-phoenix-508:MKDSN1,5/2-5,08
- added PUMP_LED: (no value), con-amp:MTA02-100
- added Q2: BC337, transistor-npn:BC337
- added R4, R5: 470, resistor-power:RRS1/8
Connections:
- new net D6: R4.2
- new net N$2: Q2.B, R4.1
- new net N$4: D2.A, PUMP-2.KL, PUMP_LED.1, Q2.C
- new net N$6: PUMP_LED.2, R5.1
- net GND: now also Q2.E
- net VIN: now also D2.C, PUMP-1.KL, R5.2
Other:
- moved on the sheet: DS18B20-1, DS18B20-2, DS18B20-3
Changed lines of the file:
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@@
 <part name="BUTTONS" library="con-amp" library_urn="urn:adsk.eagle:library:127" deviceset="MTA06-100" device="" package3d_urn="urn:adsk.eagle:package:8081635/1"/>
 <part name="HTR_LED" library="con-amp" library_urn="urn:adsk.eagle:library:127" deviceset="MTA02-100" device="" package3d_urn="urn:adsk.eagle:package:8081649/1"/>
+<part name="R4" library="resistor-power" library_urn="urn:adsk.eagle:library:344" deviceset="R" device="RS1/8" package3d_urn="urn:adsk.eagle:package:25168/1" value="470"/>
+<part name="Q2" library="transistor-npn" library_urn="urn:adsk.eagle:library:398" deviceset="BC337*" device="" package3d_urn="urn:adsk.eagle:package:28523/2"/>
+<part name="GND1" library="supply1" library_urn="urn:adsk.eagle:library:371" deviceset="GND" device=""/>
+<part name="D2" library="diode" library_urn="urn:adsk.eagle:library:210" deviceset="1N4004" device="" package3d_urn="urn:adsk.eagle:package:43336/1" value="1N4007"/>
+<part name="PUMP" library="con-phoenix-508" library_urn="urn:adsk.eagle:library:176" deviceset="MKDSN1,5/2-5,08" device="" package3d_urn="urn:adsk.eagle:package:9630/1"/>
+<part name="R5" library="resistor-power" library_urn="urn:adsk.eagle:library:344" deviceset="R" device="RS1/8" package3d_urn="urn:adsk.eagle:package:25168/1" value="470"/>
+<part name="PUMP_LED" library="con-amp" library_urn="urn:adsk.eagle:library:127" deviceset="MTA02-100" device="" package3d_urn="urn:adsk.eagle:package:8081649/1"/>
 </parts>
 <sheets>
@@
 <attribute name="VALUE" x="20.32" y="34.417" size="1.778" layer="96"/>
 </instance>
-<instance part="DS18B20" gate="-1" x="40.64" y="-38.1" smashed="yes">
-<attribute name="NAME" x="43.688" y="-38.989" size="1.778" layer="95"/>
-<attribute name="VALUE" x="38.1" y="-34.163" size="1.778" layer="96"/>
-</instance>
-<instance part="DS18B20" gate="-2" x="40.64" y="-43.18" smashed="yes">
-<attribute name="NAME" x="43.688" y="-44.069" size="1.778" layer="95"/>
-</instance>
-<instance part="DS18B20" gate="-3" x="40.64" y="-48.26" smashed="yes">
-<attribute name="NAME" x="43.688" y="-49.149" size="1.778" layer="95"/>
+<instance part="DS18B20" gate="-1" x="111.76" y="-33.02" smashed="yes">
+<attribute name="NAME" x="114.808" y="-33.909" size="1.778" layer="95"/>
+<attribute name="VALUE" x="109.22" y="-29.083" size="1.778" layer="96"/>
+</instance>
+<instance part="DS18B20" gate="-2" x="111.76" y="-38.1" smashed="yes">
+<attribute name="NAME" x="114.808" y="-38.989" size="1.778" layer="95"/>
+</instance>
+<instance part="DS18B20" gate="-3" x="111.76" y="-43.18" smashed="yes">
+<attribute name="NAME" x="114.808" y="-44.069" size="1.778" layer="95"/>
 </instance>
 <instance part="P+1" gate="VCC" x="96.52" y="5.08" smashed="yes">
@@
 <attribute name="NAME" x="27.94" y="25.4" size="1.778" layer="95"/>
 <attribute name="VALUE" x="21.59" y="25.4" size="1.778" layer="96" rot="R270"/>
+</instance>
+<instance part="R4" gate="G$1" x="-20.32" y="-2.54" smashed="yes" rot="R90">
+<attribute name="NAME" x="-21.6916" y="-6.35" size="1.778" layer="95" rot="R90"/>
+<attribute name="VALUE" x="-17.399" y="-6.35" size="1.778" layer="96" rot="R90"/>
+</instance>
+<instance part="Q2" gate="G$1" x="-20.32" y="-12.7" smashed="yes" rot="R270">
+<attribute name="NAME" x="-25.4" y="-20.32" size="1.778" layer="95"/>
+<attribute name="VALUE" x="-25.4" y="-17.78" size="1.778" layer="96"/>
+</instance>
+<instance part="GND1" gate="1" x="-38.1" y="-15.24" smashed="yes" rot="R270">
+<attribute name="VALUE" x="-40.64" y="-12.7" size="1.778" layer="96" rot="R270"/>
+</instance>
+<instance part="D2" gate="1" x="-7.62" y="-17.78" smashed="yes">
+<attribute name="NAME" x="-5.08" y="-17.2974" size="1.778" layer="95"/>
+<attribute name="VALUE" x="-5.08" y="-20.0914" size="1.778" layer="96"/>
+</instance>
+<instance part="PUMP" gate="-1" x="22.86" y="-2.54" smashed="yes">
+<attribute name="NAME" x="25.908" y="-3.429" size="1.778" layer="95"/>
+<attribute name="VALUE" x="20.32" y="-6.223" size="1.778" layer="96"/>
+</instance>
+<instance part="PUMP" gate="-2" x="22.86" y="-7.62" smashed="yes">
+<attribute name="NAME" x="25.908" y="-8.509" size="1.778" layer="95"/>
+<attribute name="VALUE" x="20.32" y="-11.303" size="1.778" layer="96"/>
+</instance>
+<instance part="R5" gate="G$1" x="10.16" y="-17.78" smashed="yes" rot="R180">
+<attribute name="NAME" x="13.97" y="-19.1516" size="1.778" layer="95" rot="R180"/>
+<attribute name="VALUE" x="13.97" y="-14.859" size="1.778" layer="96" rot="R180"/>
+</instance>
+<instance part="PUMP_LED" gate="G$1" x="25.4" y="-15.24" smashed="yes" rot="R270">
+<attribute name="NAME" x="27.94" y="-20.32" size="1.778" layer="95"/>
+<attribute name="VALUE" x="21.59" y="-20.32" size="1.778" layer="96" rot="R270"/>
 </instance>
 </instances>
@@
 <wire x1="-35.56" y1="38.1" x2="-35.56" y2="30.48" width="0.1524" layer="91"/>
 <junction x="-35.56" y="30.48"/>
+</segment>
+<segment>
+<pinref part="GND1" gate="1" pin="GND"/>
+<pinref part="Q2" gate="G$1" pin="E"/>
+<wire x1="-35.56" y1="-15.24" x2="-25.4" y2="-15.24" width="0.1524" layer="91"/>
 </segment>
 </net>
@@
 <label x="7.62" y="43.18" size="1.778" layer="95"/>
 </segment>
+<segment>
+<pinref part="D2" gate="1" pin="C"/>
+<pinref part="R5" gate="G$1" pin="2"/>
+<wire x1="-5.08" y1="-17.78" x2="5.08" y2="-17.78" width="0.1524" layer="91"/>
+<wire x1="5.08" y1="-17.78" x2="5.08" y2="-22.86" width="0.1524" layer="91"/>
+<junction x="5.08" y="-17.78"/>
+<label x="5.08" y="-25.4" size="1.778" layer="95"/>
+</segment>
+<segment>
+<pinref part="PUMP" gate="-1" pin="KL"/>
+<wire x1="20.32" y1="-2.54" x2="12.7" y2="-2.54" width="0.1524" layer="91"/>
+<label x="7.62" y="-2.54" size="1.778" layer="95"/>
+</segment>
 </net>
 <net name="N$5" class="0">
@@
 </segment>
 </net>
+<net name="N$2" class="0">
+<segment>
+<pinref part="R4" gate="G$1" pin="1"/>
+<pinref part="Q2" gate="G$1" pin="B"/>
+<wire x1="-20.32" y1="-7.62" x2="-20.32" y2="-10.16" width="0.1524" layer="91"/>
+</segment>
+</net>
+<net name="N$4" class="0">
+<segment>
+<pinref part="Q2" gate="G$1" pin="C"/>
+<pinref part="PUMP_LED" gate="G$1" pin="1"/>
+<wire x1="-15.24" y1="-15.24" x2="17.78" y2="-15.24" width="0.1524" layer="91"/>
+<wire x1="17.78" y1="-15.24" x2="22.86" y2="-15.24" width="0.1524" layer="91"/>
+<wire x1="-15.24" y1="-15.24" x2="-15.24" y2="-17.78" width="0.1524" layer="91"/>
+<junction x="-15.24" y="-15.24"/>
+<pinref part="D2" gate="1" pin="A"/>
+<wire x1="-15.24" y1="-17.78" x2="-10.16" y2="-17.78" width="0.1524" layer="91"/>
+<pinref part="PUMP" gate="-2" pin="KL"/>
+<wire x1="20.32" y1="-7.62" x2="17.78" y2="-7.62" width="0.1524" layer="91"/>
+<wire x1="17.78" y1="-7.62" x2="17.78" y2="-15.24" width="0.1524" layer="91"/>
+<junction x="17.78" y="-15.24"/>
+</segment>
+</net>
+<net name="N$6" class="0">
+<segment>
+<pinref part="R5" gate="G$1" pin="1"/>
+<pinref part="PUMP_LED" gate="G$1" pin="2"/>
+<wire x1="15.24" y1="-17.78" x2="22.86" y2="-17.78" width="0.1524" layer="91"/>
+</segment>
+</net>
+<net name="D6" class="0">
+<segment>
+<pinref part="R4" gate="G$1" pin="2"/>
+<wire x1="-20.32" y1="2.54" x2="-27.94" y2="2.54" width="0.1524" layer="91"/>
+<label x="-33.02" y="2.54" size="1.778" layer="95"/>
+</segment>
+</net>

Commit message: pwr scheme
Parts:
- added PWR: MKDSN1,5/2-5,08, con-phoenix-508:MKDSN1,5/2-5,08
Connections:
- net GND: now also PWR-2.KL
- net VIN: now also PWR-1.KL
Changed lines of the file:
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@@
 <part name="R5" library="resistor-power" library_urn="urn:adsk.eagle:library:344" deviceset="R" device="RS1/8" package3d_urn="urn:adsk.eagle:package:25168/1" value="470"/>
 <part name="PUMP_LED" library="con-amp" library_urn="urn:adsk.eagle:library:127" deviceset="MTA02-100" device="" package3d_urn="urn:adsk.eagle:package:8081649/1"/>
+<part name="PWR" library="con-phoenix-508" library_urn="urn:adsk.eagle:library:176" deviceset="MKDSN1,5/2-5,08" device="" package3d_urn="urn:adsk.eagle:package:9630/1"/>
+<part name="GND2" library="supply1" library_urn="urn:adsk.eagle:library:371" deviceset="GND" device=""/>
 </parts>
 <sheets>
@@
 <attribute name="VALUE" x="21.59" y="-20.32" size="1.778" layer="96" rot="R270"/>
 </instance>
+<instance part="PWR" gate="-1" x="-22.86" y="-43.18" smashed="yes">
+<attribute name="NAME" x="-19.812" y="-44.069" size="1.778" layer="95"/>
+<attribute name="VALUE" x="-25.4" y="-46.863" size="1.778" layer="96"/>
+</instance>
+<instance part="PWR" gate="-2" x="-22.86" y="-48.26" smashed="yes">
+<attribute name="NAME" x="-19.812" y="-49.149" size="1.778" layer="95"/>
+<attribute name="VALUE" x="-25.4" y="-51.943" size="1.778" layer="96"/>
+</instance>
+<instance part="GND2" gate="1" x="-38.1" y="-48.26" smashed="yes" rot="R270">
+<attribute name="VALUE" x="-40.64" y="-45.72" size="1.778" layer="96" rot="R270"/>
+</instance>
 </instances>
 <busses>
@@
 <pinref part="Q2" gate="G$1" pin="E"/>
 <wire x1="-35.56" y1="-15.24" x2="-25.4" y2="-15.24" width="0.1524" layer="91"/>
+</segment>
+<segment>
+<pinref part="GND2" gate="1" pin="GND"/>
+<pinref part="PWR" gate="-2" pin="KL"/>
+<wire x1="-35.56" y1="-48.26" x2="-25.4" y2="-48.26" width="0.1524" layer="91"/>
 </segment>
 </net>
@@
 <label x="7.62" y="-2.54" size="1.778" layer="95"/>
 </segment>
+<segment>
+<pinref part="PWR" gate="-1" pin="KL"/>
+<wire x1="-25.4" y1="-43.18" x2="-35.56" y2="-43.18" width="0.1524" layer="91"/>
+<label x="-40.64" y="-43.18" size="1.778" layer="95"/>
+</segment>
 </net>

Commit message: display scheme
Parts:
- added LCD: LCD-HD447804-HOLES20X4-4HOLES, HD44780LCD:LCD-HD447804-HOLES20X4-4HOLES
- added R6: 470, resistor-power:RRS1/8
Connections:
- new net A4: LCD.RS
- new net A5: LCD.E
- new net D2: LCD.DB4
- new net D3: LCD.DB5
- new net D4: LCD.DB6
- new net D5: LCD.DB7
- new net N$14: LCD.A, R6.1
- new net N$7: LCD.VO, V1.S
- new net VCC: LCD.VDD, R6.2, V1.E
- net GND: now also LCD.DB0, LCD.DB1, LCD.DB2, LCD.DB3, LCD.K, LCD.R/W, LCD.VSS, V1.A
Other:
- moved on the sheet: BUTTONS, DS18B20-1, DS18B20-2, DS18B20-3, V1

Commit message: ajustando valor do registor do display scheme
Parts:
- added PUMP_LED1: (no value), con-amp:MTA02-100
- added Q3: BC337, transistor-npn:BC337
- added R7: 470, resistor-power:RRS1/8
- R6: value 470 -> 220
Changed lines of the file:
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@@
 <part name="GND2" library="supply1" library_urn="urn:adsk.eagle:library:371" deviceset="GND" device=""/>
 <part name="LCD" library="HD44780LCD" deviceset="LCD-HD44780" device="20X4-4HOLES" technology="4-HOLES"/>
-<part name="R6" library="resistor-power" library_urn="urn:adsk.eagle:library:344" deviceset="R" device="RS1/8" package3d_urn="urn:adsk.eagle:package:25168/1" value="470"/>
+<part name="R6" library="resistor-power" library_urn="urn:adsk.eagle:library:344" deviceset="R" device="RS1/8" package3d_urn="urn:adsk.eagle:package:25168/1" value="220"/>
 <part name="GND3" library="supply1" library_urn="urn:adsk.eagle:library:371" deviceset="GND" device=""/>
 <part name="P+2" library="supply1" library_urn="urn:adsk.eagle:library:371" deviceset="VCC" device="" value="+5V"/>
@@
 <part name="GND5" library="supply1" library_urn="urn:adsk.eagle:library:371" deviceset="GND" device=""/>
 <part name="P+4" library="supply1" library_urn="urn:adsk.eagle:library:371" deviceset="VCC" device="" value="+5V"/>
+<part name="PUMP_LED1" library="con-amp" library_urn="urn:adsk.eagle:library:127" deviceset="MTA02-100" device="" package3d_urn="urn:adsk.eagle:package:8081649/1"/>
+<part name="Q3" library="transistor-npn" library_urn="urn:adsk.eagle:library:398" deviceset="BC337*" device="" package3d_urn="urn:adsk.eagle:package:28523/2"/>
+<part name="R7" library="resistor-power" library_urn="urn:adsk.eagle:library:344" deviceset="R" device="RS1/8" package3d_urn="urn:adsk.eagle:package:25168/1" value="470"/>
 </parts>
 <sheets>
@@
 <attribute name="VALUE" x="76.2" y="15.24" size="1.778" layer="96" rot="R180"/>
 </instance>
+<instance part="PUMP_LED1" gate="G$1" x="78.74" y="-25.4" smashed="yes" rot="R270">
+<attribute name="NAME" x="81.28" y="-30.48" size="1.778" layer="95"/>
+<attribute name="VALUE" x="74.93" y="-30.48" size="1.778" layer="96" rot="R270"/>
+</instance>
+<instance part="Q3" gate="G$1" x="60.96" y="-33.02" smashed="yes" rot="R270">
+<attribute name="NAME" x="55.88" y="-40.64" size="1.778" layer="95"/>
+<attribute name="VALUE" x="55.88" y="-38.1" size="1.778" layer="96"/>
+</instance>
+<instance part="R7" gate="G$1" x="60.96" y="-22.86" smashed="yes" rot="R180">
+<attribute name="NAME" x="64.77" y="-24.2316" size="1.778" layer="95" rot="R180"/>
+<attribute name="VALUE" x="64.77" y="-19.939" size="1.778" layer="96" rot="R180"/>
+</instance>
 </instances>

Commit message: buzzer scheme
Parts:
- removed PUMP_LED1: (no value), con-amp:MTA02-100
- added BUZZ: (no value), con-amp:MTA02-100
Connections:
- new net D10: R7.2
- new net N$8: Q3.B, R7.1
- new net N$9: BUZZ.2, Q3.C
- net GND: now also Q3.E
- net VIN: now also BUZZ.1
Other:
- moved on the sheet: Q3, R7
Changed lines of the file:
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@@
 <part name="GND5" library="supply1" library_urn="urn:adsk.eagle:library:371" deviceset="GND" device=""/>
 <part name="P+4" library="supply1" library_urn="urn:adsk.eagle:library:371" deviceset="VCC" device="" value="+5V"/>
-<part name="PUMP_LED1" library="con-amp" library_urn="urn:adsk.eagle:library:127" deviceset="MTA02-100" device="" package3d_urn="urn:adsk.eagle:package:8081649/1"/>
+<part name="BUZZ" library="con-amp" library_urn="urn:adsk.eagle:library:127" deviceset="MTA02-100" device="" package3d_urn="urn:adsk.eagle:package:8081649/1"/>
 <part name="Q3" library="transistor-npn" library_urn="urn:adsk.eagle:library:398" deviceset="BC337*" device="" package3d_urn="urn:adsk.eagle:package:28523/2"/>
 <part name="R7" library="resistor-power" library_urn="urn:adsk.eagle:library:344" deviceset="R" device="RS1/8" package3d_urn="urn:adsk.eagle:package:25168/1" value="470"/>
+<part name="GND6" library="supply1" library_urn="urn:adsk.eagle:library:371" deviceset="GND" device=""/>
 </parts>
 <sheets>
@@
 <attribute name="VALUE" x="76.2" y="15.24" size="1.778" layer="96" rot="R180"/>
 </instance>
-<instance part="PUMP_LED1" gate="G$1" x="78.74" y="-25.4" smashed="yes" rot="R270">
-<attribute name="NAME" x="81.28" y="-30.48" size="1.778" layer="95"/>
-<attribute name="VALUE" x="74.93" y="-30.48" size="1.778" layer="96" rot="R270"/>
-</instance>
-<instance part="Q3" gate="G$1" x="60.96" y="-33.02" smashed="yes" rot="R270">
-<attribute name="NAME" x="55.88" y="-40.64" size="1.778" layer="95"/>
-<attribute name="VALUE" x="55.88" y="-38.1" size="1.778" layer="96"/>
-</instance>
-<instance part="R7" gate="G$1" x="60.96" y="-22.86" smashed="yes" rot="R180">
-<attribute name="NAME" x="64.77" y="-24.2316" size="1.778" layer="95" rot="R180"/>
-<attribute name="VALUE" x="64.77" y="-19.939" size="1.778" layer="96" rot="R180"/>
+<instance part="BUZZ" gate="G$1" x="116.84" y="-12.7" smashed="yes" rot="R270">
+<attribute name="NAME" x="119.38" y="-17.78" size="1.778" layer="95"/>
+<attribute name="VALUE" x="113.03" y="-17.78" size="1.778" layer="96" rot="R270"/>
+</instance>
+<instance part="Q3" gate="G$1" x="99.06" y="-12.7" smashed="yes" rot="R270">
+<attribute name="NAME" x="93.98" y="-20.32" size="1.778" layer="95"/>
+<attribute name="VALUE" x="93.98" y="-17.78" size="1.778" layer="96"/>
+</instance>
+<instance part="R7" gate="G$1" x="91.44" y="-7.62" smashed="yes" rot="R180">
+<attribute name="NAME" x="95.25" y="-8.9916" size="1.778" layer="95" rot="R180"/>
+<attribute name="VALUE" x="95.25" y="-4.699" size="1.778" layer="96" rot="R180"/>
+</instance>
+<instance part="GND6" gate="1" x="88.9" y="-15.24" smashed="yes" rot="R270">
+<attribute name="VALUE" x="86.36" y="-12.7" size="1.778" layer="96" rot="R270"/>
 </instance>
 </instances>
@@
 <wire x1="88.9" y1="17.78" x2="91.44" y2="17.78" width="0.1524" layer="91"/>
 </segment>
+<segment>
+<pinref part="GND6" gate="1" pin="GND"/>
+<pinref part="Q3" gate="G$1" pin="E"/>
+<wire x1="91.44" y1="-15.24" x2="93.98" y2="-15.24" width="0.1524" layer="91"/>
+</segment>
 </net>
 <net name="N$1" class="0">
@@
 <label x="-40.64" y="-43.18" size="1.778" layer="95"/>
 </segment>
+<segment>
+<pinref part="BUZZ" gate="G$1" pin="1"/>
+<wire x1="114.3" y1="-12.7" x2="111.76" y2="-12.7" width="0.1524" layer="91"/>
+<label x="106.68" y="-12.7" size="1.778" layer="95"/>
+</segment>
 </net>
 <net name="N$5" class="0">
@@
 </segment>
 </net>
+<net name="N$8" class="0">
+<segment>
+<pinref part="Q3" gate="G$1" pin="B"/>
+<pinref part="R7" gate="G$1" pin="1"/>
+<wire x1="99.06" y1="-10.16" x2="99.06" y2="-7.62" width="0.1524" layer="91"/>
+<wire x1="99.06" y1="-7.62" x2="96.52" y2="-7.62" width="0.1524" layer="91"/>
+</segment>
+</net>
+<net name="N$9" class="0">
+<segment>
+<pinref part="Q3" gate="G$1" pin="C"/>
+<pinref part="BUZZ" gate="G$1" pin="2"/>
+<wire x1="104.14" y1="-15.24" x2="114.3" y2="-15.24" width="0.1524" layer="91"/>
+</segment>
+</net>
+<net name="D10" class="0">
+<segment>
+<pinref part="R7" gate="G$1" pin="2"/>
+<wire x1="86.36" y1="-7.62" x2="83.82" y2="-7.62" width="0.1524" layer="91"/>
+<label x="78.74" y="-7.62" size="1.778" layer="95"/>
+</segment>
+</net>

Commit message: rst scheme
Parts:
- added RST: (no value), con-amp:MTA02-100
Connections:
- new net RST: RST.2
- net GND: now also RST.1
Changed lines of the file:
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@@
 <part name="R7" library="resistor-power" library_urn="urn:adsk.eagle:library:344" deviceset="R" device="RS1/8" package3d_urn="urn:adsk.eagle:package:25168/1" value="470"/>
 <part name="GND6" library="supply1" library_urn="urn:adsk.eagle:library:371" deviceset="GND" device=""/>
+<part name="RST" library="con-amp" library_urn="urn:adsk.eagle:library:127" deviceset="MTA02-100" device="" package3d_urn="urn:adsk.eagle:package:8081649/1"/>
+<part name="GND7" library="supply1" library_urn="urn:adsk.eagle:library:371" deviceset="GND" device=""/>
 </parts>
 <sheets>
@@
 <instance part="GND6" gate="1" x="88.9" y="-15.24" smashed="yes" rot="R270">
 <attribute name="VALUE" x="86.36" y="-12.7" size="1.778" layer="96" rot="R270"/>
+</instance>
+<instance part="RST" gate="G$1" x="104.14" y="-43.18" smashed="yes" rot="R270">
+<attribute name="NAME" x="106.68" y="-48.26" size="1.778" layer="95"/>
+<attribute name="VALUE" x="100.33" y="-48.26" size="1.778" layer="96" rot="R270"/>
+</instance>
+<instance part="GND7" gate="1" x="91.44" y="-43.18" smashed="yes" rot="R270">
+<attribute name="VALUE" x="88.9" y="-40.64" size="1.778" layer="96" rot="R270"/>
 </instance>
 </instances>
@@
 <wire x1="91.44" y1="-15.24" x2="93.98" y2="-15.24" width="0.1524" layer="91"/>
 </segment>
+<segment>
+<pinref part="GND7" gate="1" pin="GND"/>
+<pinref part="RST" gate="G$1" pin="1"/>
+<wire x1="93.98" y1="-43.18" x2="101.6" y2="-43.18" width="0.1524" layer="91"/>
+</segment>
 </net>
 <net name="N$1" class="0">
@@
 </segment>
 </net>
+<net name="RST" class="0">
+<segment>
+<pinref part="RST" gate="G$1" pin="2"/>
+<wire x1="101.6" y1="-45.72" x2="99.06" y2="-45.72" width="0.1524" layer="91"/>
+<label x="93.98" y="-45.72" size="1.778" layer="95"/>
+</segment>
+</net>
