File: atividades/atividade-03/controlador_temperatura.brd (EAGLE design)
At the start: 160 x 100 mm, 34 parts, among them Q1 BC337, Q2 BC337, Q3 BC337

Commit message: abrindo circuito
Parts:
- removed SV1, SV2: (no value), con-lstb:MA08-1
- added DISPLAY: DCS, con-panduit:057-016-1
- added SHIELD: SCD, con-panduit:057-016-1
- LCD: value LCD-HD447804-HOLES20X4-4HOLES -> TUXGR_16X2_R2; device HD44780LCD:LCD-20X4-4HOLES -> display-lcd:TUXGR_16X2_R2
- moved R11 81.3 mm to (-17.8, 82.5)
- moved Q3 76.2 mm to (-22.9, 100.3)
- moved HTR_LED 62.5 mm to (-92.7, 82.5)
- moved PUMP_LED 62.5 mm to (-82.5, 82.5)
- moved LCD 61.1 mm to (-53.3, 19.1)
- moved D1 33.6 mm to (-39.4, 82.5)
- moved D2 33.6 mm to (-52.1, 82.5)
- moved BUTTONS 33.6 mm to (-66.0, 82.5)
- moved RST 22.5 mm to (-22.9, 90.2)
- moved SHIELD_ARDUINO_CB2 22.5 mm to (-68.6, 88.9)
- moved BUZZ 22.5 mm to (-16.5, 90.2)
- moved SHIELD_ARDUINO_CB1 22.5 mm to (-43.2, 88.9)
- moved HTR 21.6 mm to (-20.3, 44.5)
- moved PUMP 21.6 mm to (-34.3, 44.5)
- moved PWR 21.6 mm to (-48.3, 44.5)
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Connections:
- removed net A: LCD.P$15, R6.1, SV2.7
- removed net VO: LCD.P$3, SV1.3, V1.S
- new net N$10: DISPLAY.2, LCD.2
- new net N$11: DISPLAY.3, LCD.3
- new net N$12: DISPLAY.4, LCD.4
- new net N$13: DISPLAY.5, LCD.5
- new net N$14: DISPLAY.6, LCD.6
- new net N$15: DISPLAY.7, LCD.7
- new net N$16: DISPLAY.8, LCD.8
- new net N$17: DISPLAY.9, LCD.9
- new net N$18: DISPLAY.10, LCD.10
- new net N$19: DISPLAY.11, LCD.11
- new net N$20: DISPLAY.12, LCD.12
- new net N$21: DISPLAY.13, LCD.13
- new net N$22: DISPLAY.14, LCD.14
- new net N$23: DISPLAY.15, LCD.15
- new net N$24: DISPLAY.16, LCD.16
- new net N$25: R6.1, SHIELD.15
- new net N$26: SHIELD.3, V1.S
- new net N$7: DISPLAY.1, LCD.1
- net A4: now also SHIELD.4; no longer LCD.P$4, SV1.4
- net A5: now also SHIELD.6; no longer LCD.P$6, SV1.6
- net D2: now also SHIELD.11; no longer LCD.P$11, SV2.3
- net D3: now also SHIELD.12; no longer LCD.P$12, SV2.4
- net D4: now also SHIELD.13; no longer LCD.P$13, SV2.5
- net D5: now also SHIELD.14; no longer LCD.P$14, SV2.6
- net GND: now also SHIELD.1, SHIELD.10, SHIELD.16, SHIELD.5, SHIELD.7, SHIELD.8, SHIELD.9; no longer LCD.P$1, LCD.P$10, LCD.P$16, LCD.P$5, LCD.P$7, LCD.P$8, LCD.P$9, SV1.1, SV1.5, SV1.7, SV1.8, SV2.1, SV2.2, SV2.8
- net VCC: now also SHIELD.2; no longer LCD.P$2, SV1.2
